File: Schaltmischer/Schaltmischer.sch (KiCad schematic (older format))
At the start: 13 parts

Commit message: Schaltplan Rev B
Parts:
- added P?: IN, symbol CONN_01X02
- added P?: OUT, symbol CONN_01X02
- added P?: Takt, symbol CONN_01X03
- added P?: Power, symbol CONN_01X02
- T1, T2: renamed from T?; value TRANSFORMER_1P_2S -> Übertrager
- gave numbers to parts that had none: 7
Connections:
- net +5V: now also P?.1 (P1)
- net GND: now also P?.2 (P2), P?.2 (P2), P?.2 (P2), P?.2 (P2)
- net IN1: no longer U1.1 (OE)
- net IN: now reaches T1.1 (AA)
- net IN: now also P?.1 (P1)
- net OUT: now reaches T2.1 (AA)
- net OUT: now also P?.1 (P1)
- net IN2 renamed SW2
- net SW2: now also P?.3 (P3)
- new net SW1: P?.1 (P1), U1.1 (OE)
Other:
- moved on the sheet: C1, C2, C3, C4, R1, R2, T1, T2, U1A, U1B, U1C, U1D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

Commit message: Schaltplan Rev B
Parts:
- gave numbers to parts that had none: 4
Changed lines of the file:
@@
 	8200 4400 8300 4400
 $Comp
-L GND #PWR01
+L GND #PWR5
 U 1 1 5AD25ECC
 P 2500 4700
-F 0 "#PWR01" H 2500 4450 50  0001 C CNN
+F 0 "#PWR5" H 2500 4450 50  0001 C CNN
 F 1 "GND" H 2500 4550 50  0000 C CNN
 F 2 "" H 2500 4700 50  0000 C CNN
@@
 $EndComp
 $Comp
-L GND #PWR02
+L GND #PWR11
 U 1 1 5AD25F11
 P 9300 4700
-F 0 "#PWR02" H 9300 4450 50  0001 C CNN
+F 0 "#PWR11" H 9300 4450 50  0001 C CNN
 F 1 "GND" H 9300 4550 50  0000 C CNN
 F 2 "" H 9300 4700 50  0000 C CNN
@@
 Connection ~ 3600 4300
 $Comp
-L GND #PWR03
+L GND #PWR9
 U 1 1 5AD27FC4
 P 3800 5400
-F 0 "#PWR03" H 3800 5150 50  0001 C CNN
+F 0 "#PWR9" H 3800 5150 50  0001 C CNN
 F 1 "GND" H 3800 5250 50  0000 C CNN
 F 2 "" H 3800 5400 50  0000 C CNN
@@
 $EndComp
 $Comp
-L GND #PWR04
+L GND #PWR10
 U 1 1 5AD283A9
 P 8000 5400
-F 0 "#PWR04" H 8000 5150 50  0001 C CNN
+F 0 "#PWR10" H 8000 5150 50  0001 C CNN
 F 1 "GND" H 8000 5250 50  0000 C CNN
 F 2 "" H 8000 5400 50  0000 C CNN
@@
 Connection ~ 3200 1800
 $Comp
-L GND #PWR05
+L GND #PWR6
 U 1 1 5AD2A7C7
 P 2600 2500
-F 0 "#PWR05" H 2600 2250 50  0001 C CNN
+F 0 "#PWR6" H 2600 2250 50  0001 C CNN
 F 1 "GND" H 2600 2350 50  0000 C CNN
 F 2 "" H 2600 2500 50  0000 C CNN
@@
 $EndComp
 $Comp
-L GND #PWR06
+L GND #PWR8
 U 1 1 5AD2A809
 P 3200 2500
-F 0 "#PWR06" H 3200 2250 50  0001 C CNN
+F 0 "#PWR8" H 3200 2250 50  0001 C CNN
 F 1 "GND" H 3200 2350 50  0000 C CNN
 F 2 "" H 3200 2500 50  0000 C CNN
@@
 Connection ~ 2900 1800
 $Comp
-L +5V #PWR07
+L +5V #PWR7
 U 1 1 5AD2B086
 P 2900 1100
-F 0 "#PWR07" H 2900 950 50  0001 C CNN
+F 0 "#PWR7" H 2900 950 50  0001 C CNN
 F 1 "+5V" H 2900 1240 50  0000 C CNN
 F 2 "" H 2900 1100 50  0000 C CNN
@@
 	2900 1100 2900 1200
 $Comp
-L GND #PWR08
+L GND #PWR13
 U 1 1 5AD2BFA4
 P 9700 2700
-F 0 "#PWR08" H 9700 2450 50  0001 C CNN
+F 0 "#PWR13" H 9700 2450 50  0001 C CNN
 F 1 "GND" H 9700 2550 50  0000 C CNN
 F 2 "" H 9700 2700 50  0000 C CNN
@@
 $EndComp
 $Comp
-L +5V #PWR09
+L +5V #PWR12
 U 1 1 5AD2C04B
 P 9700 1300
-F 0 "#PWR09" H 9700 1150 50  0001 C CNN
+F 0 "#PWR12" H 9700 1150 50  0001 C CNN
 F 1 "+5V" H 9700 1440 50  0000 C CNN
 F 2 "" H 9700 1300 50  0000 C CNN
@@
 OUT
 $Comp
-L CONN_01X02 P?
+L CONN_01X02 P2
 U 1 1 5AD2F4C3
 P 1200 4350
-F 0 "P?" H 1200 4500 50  0000 C CNN
+F 0 "P2" H 1200 4500 50  0000 C CNN
 F 1 "IN" V 1300 4350 50  0000 C CNN
 F 2 "" H 1200 4350 50  0000 C CNN
@@
 	1500 4400 1500 4500
 $Comp
-L GND #PWR?
+L GND #PWR3
 U 1 1 5AD2F7B4
 P 1500 4500
-F 0 "#PWR?" H 1500 4250 50  0001 C CNN
+F 0 "#PWR3" H 1500 4250 50  0001 C CNN
 F 1 "GND" H 1500 4350 50  0000 C CNN
 F 2 "" H 1500 4500 50  0000 C CNN
@@
 $EndComp
 $Comp
-L CONN_01X02 P?
+L CONN_01X02 P4
 U 1 1 5AD30156
 P 10700 4350
-F 0 "P?" H 10700 4500 50  0000 C CNN
+F 0 "P4" H 10700 4500 50  0000 C CNN
 F 1 "OUT" V 10800 4350 50  0000 C CNN
 F 2 "" H 10700 4350 50  0000 C CNN
@@
 OUT
 $Comp
-L GND #PWR?
+L GND #PWR14
 U 1 1 5AD30334
 P 10400 4500
-F 0 "#PWR?" H 10400 4250 50  0001 C CNN
+F 0 "#PWR14" H 10400 4250 50  0001 C CNN
 F 1 "GND" H 10400 4350 50  0000 C CNN
 F 2 "" H 10400 4500 50  0000 C CNN
@@
 	10400 4200 10300 4200
 $Comp
-L CONN_01X03 P?
+L CONN_01X03 P3
 U 1 1 5AD310CD
 P 1200 5800
-F 0 "P?" H 1200 6000 50  0000 C CNN
+F 0 "P3" H 1200 6000 50  0000 C CNN
 F 1 "Takt" V 1300 5800 50  0000 C CNN
 F 2 "" H 1200 5800 50  0000 C CNN
@@
 $EndComp
 $Comp
-L GND #PWR?
+L GND #PWR4
 U 1 1 5AD31244
 P 1600 6100
-F 0 "#PWR?" H 1600 5850 50  0001 C CNN
+F 0 "#PWR4" H 1600 5850 50  0001 C CNN
 F 1 "GND" H 1600 5950 50  0000 C CNN
 F 2 "" H 1600 6100 50  0000 C CNN
@@
 	1400 5700 1800 5700
 $Comp
-L CONN_01X02 P?
+L CONN_01X02 P1
 U 1 1 5AD3295E
 P 1200 1750
-F 0 "P?" H 1200 1900 50  0000 C CNN
+F 0 "P1" H 1200 1900 50  0000 C CNN
 F 1 "Power" V 1300 1750 50  0000 C CNN
 F 2 "" H 1200 1750 50  0000 C CNN
@@
 $EndComp
 $Comp
-L GND #PWR?
+L GND #PWR2
 U 1 1 5AD32AD2
 P 1500 1900
-F 0 "#PWR?" H 1500 1650 50  0001 C CNN
+F 0 "#PWR2" H 1500 1650 50  0001 C CNN
 F 1 "GND" H 1500 1750 50  0000 C CNN
 F 2 "" H 1500 1900 50  0000 C CNN
@@
 	1500 1800 1500 1900
 $Comp
-L +5V #PWR?
+L +5V #PWR1
 U 1 1 5AD32D6F
 P 1500 1600
-F 0 "#PWR?" H 1500 1450 50  0001 C CNN
+F 0 "#PWR1" H 1500 1450 50  0001 C CNN
 F 1 "+5V" H 1500 1740 50  0000 C CNN
 F 2 "" H 1500 1600 50  0000 C CNN

Commit message: Schaltplan Rev C
Parts:
- C1: footprint (none) -> Capacitors_THT:C_Radial_D6.3_L11.2_P2.5
- C2, C3, C4: footprint (none) -> Capacitors_SMD:C_1206_HandSoldering
- P1, P2, P4: footprint (none) -> Pin_Headers:Pin_Header_Straight_1x02_Pitch2.54mm
- P3: footprint (none) -> Pin_Headers:Pin_Header_Straight_1x03_Pitch2.54mm
- R1, R2: footprint (none) -> Resistors_SMD:R_1206_HandSoldering
- T1, T2: footprint (none) -> HF_Transformers:T-622; symbol TRANSFORMER_1P_2S -> TRANSFORMER_1P_2S_2
- U1: footprint (none) -> Housings_SOIC:SOIC-14_3.9x8.7mm_Pitch1.27mm
Connections:
- net GND: now also T1.6 (AB), T2.6 (AB); no longer T1.2 (AB), T2.2 (AB)
- net at U1.11 (B), U1.6 (B): now also T2.5 (SD); no longer T2.6 (SD)
- net at U1.12 (A), U1.9 (A): now also T1.5 (SD); no longer T1.6 (SD)
- net at C1.1, C2.1, C3.1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: now also T1.2 (SC), T2.2 (SC); no longer T1.5 (SC), T2.5 (SC)
Changed lines of the file:
@@
 LIBS:contrib
 LIBS:valves
+LIBS:Schaltmischer-cache
 EELAYER 25 0
 EELAYER END
@@
 Title "Schaltmischer"
 Date "2018-04-14"
-Rev "B"
+Rev "C"
 Comp "Jonas Gappert"
 Comment1 ""
@@
 F 0 "U1" H 5500 2650 60  0000 C CNN
 F 1 "FST3125" H 5600 1950 60  0000 C CNN
-F 2 "" H 5500 2400 60  0001 C CNN
+F 2 "Housings_SOIC:SOIC-14_3.9x8.7mm_Pitch1.27mm" H 5500 2400 60  0001 C CNN
 F 3 "" H 5500 2400 60  0001 C CNN
 	1    5500 2400
@@
 F 0 "U1" H 5500 3650 60  0000 C CNN
 F 1 "FST3125" H 5600 2950 60  0000 C CNN
-F 2 "" H 5500 3400 60  0001 C CNN
+F 2 "Housings_SOIC:SOIC-14_3.9x8.7mm_Pitch1.27mm" H 5500 3400 60  0001 C CNN
 F 3 "" H 5500 3400 60  0001 C CNN
 	2    5500 3400
@@
 F 0 "U1" H 5500 4850 60  0000 C CNN
 F 1 "FST3125" H 5600 4150 60  0000 C CNN
-F 2 "" H 5500 4600 60  0001 C CNN
+F 2 "Housings_SOIC:SOIC-14_3.9x8.7mm_Pitch1.27mm" H 5500 4600 60  0001 C CNN
 F 3 "" H 5500 4600 60  0001 C CNN
 	3    5500 4600
@@
 F 0 "U1" H 5500 5850 60  0000 C CNN
 F 1 "FST3125" H 5600 5150 60  0000 C CNN
-F 2 "" H 5500 5600 60  0001 C CNN
+F 2 "Housings_SOIC:SOIC-14_3.9x8.7mm_Pitch1.27mm" H 5500 5600 60  0001 C CNN
 F 3 "" H 5500 5600 60  0001 C CNN
 	4    5500 5600
@@
 F 0 "U1" H 9300 2150 60  0000 C CNN
 F 1 "FST3125" H 9400 1450 60  0000 C CNN
-F 2 "" H 9300 1900 60  0001 C CNN
+F 2 "Housings_SOIC:SOIC-14_3.9x8.7mm_Pitch1.27mm" H 9300 1900 60  0001 C CNN
 F 3 "" H 9300 1900 60  0001 C CNN
 	5    9300 1900
@@
 	6600 5900 6300 5900
 $Comp
-L TRANSFORMER_1P_2S T1
-U 1 1 5AD259DF
-P 3100 4300
-F 0 "T1" H 3100 4800 50  0000 C CNN
-F 1 "Übertrager" H 3100 3800 50  0000 C CNN
-F 2 "" H 3100 4300 50  0000 C CNN
-F 3 "" H 3100 4300 50  0000 C CNN
-	1    3100 4300
-	1    0    0    -1
-$EndComp
-$Comp
-L TRANSFORMER_1P_2S T2
+L TRANSFORMER_1P_2S_2 T2
 U 1 1 5AD25A86
 P 8700 4300
 F 0 "T2" H 8700 4800 50  0000 C CNN
 F 1 "Übertrager" H 8700 3800 50  0000 C CNN
-F 2 "" H 8700 4300 50  0000 C CNN
+F 2 "HF_Transformers:T-622" H 8700 4300 50  0001 C CNN
 F 3 "" H 8700 4300 50  0000 C CNN
 	1    8700 4300
@@
 	8200 4400 8300 4400
 $Comp
-L GND #PWR5
+L GND #PWR01
 U 1 1 5AD25ECC
 P 2500 4700
-F 0 "#PWR5" H 2500 4450 50  0001 C CNN
+F 0 "#PWR01" H 2500 4450 50  0001 C CNN
 F 1 "GND" H 2500 4550 50  0000 C CNN
 F 2 "" H 2500 4700 50  0000 C CNN
@@
 $EndComp
 $Comp
-L GND #PWR11
+L GND #PWR02
 U 1 1 5AD25F11
 P 9300 4700
-F 0 "#PWR11" H 9300 4450 50  0001 C CNN
+F 0 "#PWR02" H 9300 4450 50  0001 C CNN
 F 1 "GND" H 9300 4550 50  0000 C CNN
 F 2 "" H 9300 4700 50  0000 C CNN
@@
 F 0 "C2" H 3825 5250 50  0000 L CNN
 F 1 "10n" H 3825 5050 50  0000 L CNN
-F 2 "" H 3838 5000 50  0000 C CNN
+F 2 "Capacitors_SMD:C_1206_HandSoldering" H 3838 5000 50  0001 C CNN
 F 3 "" H 3800 5150 50  0000 C CNN
 	1    3800 5150
@@
 Connection ~ 3600 4300
 $Comp
-L GND #PWR9
+L GND #PWR03
 U 1 1 5AD27FC4
 P 3800 5400
-F 0 "#PWR9" H 3800 5150 50  0001 C CNN
+F 0 "#PWR03" H 3800 5150 50  0001 C CNN
 F 1 "GND" H 3800 5250 50  0000 C CNN
 F 2 "" H 3800 5400 50  0000 C CNN
@@
 F 0 "C3" H 8025 5250 50  0000 L CNN
 F 1 "10n" H 8025 5050 50  0000 L CNN
-F 2 "" H 8038 5000 50  0000 C CNN
+F 2 "Capacitors_SMD:C_1206_HandSoldering" H 8038 5000 50  0001 C CNN
 F 3 "" H 8000 5150 50  0000 C CNN
 	1    8000 5150
@@
 $EndComp
 $Comp
-L GND #PWR10
+L GND #PWR04
 U 1 1 5AD283A9
 P 8000 5400
-F 0 "#PWR10" H 8000 5150 50  0001 C CNN
+F 0 "#PWR04" H 8000 5150 50  0001 C CNN
 F 1 "GND" H 8000 5250 50  0000 C CNN
 F 2 "" H 8000 5400 50  0000 C CNN
@@
 F 0 "C1" H 3225 2350 50  0000 L CNN
 F 1 "10µ" H 3225 2150 50  0000 L CNN
-F 2 "" H 3238 2100 50  0000 C CNN
+F 2 "Capacitors_THT:C_Radial_D6.3_L11.2_P2.5" H 3238 2100 50  0001 C CNN
 F 3 "" H 3200 2250 50  0000 C CNN
 	1    3200 2250
@@
 F 0 "R1" V 2680 2250 50  0000 C CNN
 F 1 "1k5" V 2600 2250 50  0000 C CNN
-F 2 "" V 2530 2250 50  0000 C CNN
+F 2 "Resistors_SMD:R_1206_HandSoldering" V 2530 2250 50  0001 C CNN
 F 3 "" H 2600 2250 50  0000 C CNN
 	1    2600 2250
@@
 Connection ~ 3200 1800
 $Comp
-L GND #PWR6
+L GND #PWR05
 U 1 1 5AD2A7C7
 P 2600 2500
-F 0 "#PWR6" H 2600 2250 50  0001 C CNN
+F 0 "#PWR05" H 2600 2250 50  0001 C CNN
 F 1 "GND" H 2600 2350 50  0000 C CNN
 F 2 "" H 2600 2500 50  0000 C CNN
@@
 $EndComp
 $Comp
-L GND #PWR8
+L GND #PWR06
 U 1 1 5AD2A809
 P 3200 2500
-F 0 "#PWR8" H 3200 2250 50  0001 C CNN
+F 0 "#PWR06" H 3200 2250 50  0001 C CNN
 F 1 "GND" H 3200 2350 50  0000 C CNN
 F 2 "" H 3200 2500 50  0000 C CNN
@@
 F 0 "R2" V 2980 1350 50  0000 C CNN
 F 1 "3k3" V 2900 1350 50  0000 C CNN
-F 2 "" V 2830 1350 50  0000 C CNN
+F 2 "Resistors_SMD:R_1206_HandSoldering" V 2830 1350 50  0001 C CNN
 F 3 "" H 2900 1350 50  0000 C CNN
 	1    2900 1350
@@
 Connection ~ 2900 1800
 $Comp
-L +5V #PWR7
+L +5V #PWR07
 U 1 1 5AD2B086
 P 2900 1100
-F 0 "#PWR7" H 2900 950 50  0001 C CNN
+F 0 "#PWR07" H 2900 950 50  0001 C CNN
 F 1 "+5V" H 2900 1240 50  0000 C CNN
 F 2 "" H 2900 1100 50  0000 C CNN
@@
 	2900 1100 2900 1200
 $Comp
-L GND #PWR13
+L GND #PWR08
 U 1 1 5AD2BFA4
 P 9700 2700
-F 0 "#PWR13" H 9700 2450 50  0001 C CNN
+F 0 "#PWR08" H 9700 2450 50  0001 C CNN
 F 1 "GND" H 9700 2550 50  0000 C CNN
 F 2 "" H 9700 2700 50  0000 C CNN
@@
 $EndComp
 $Comp
-L +5V #PWR12
+L +5V #PWR09
 U 1 1 5AD2C04B
 P 9700 1300
-F 0 "#PWR12" H 9700 1150 50  0001 C CNN
+F 0 "#PWR09" H 9700 1150 50  0001 C CNN
 F 1 "+5V" H 9700 1440 50  0000 C CNN
 F 2 "" H 9700 1300 50  0000 C CNN
@@
 F 0 "C4" H 10225 2050 50  0000 L CNN
 F 1 "100n" H 10225 1850 50  0000 L CNN
-F 2 "" H 10238 1800 50  0000 C CNN
+F 2 "Capacitors_SMD:C_1206_HandSoldering" H 10238 1800 50  0001 C CNN
 F 3 "" H 10200 1950 50  0000 C CNN
 	1    10200 1950
@@
 F 0 "P2" H 1200 4500 50  0000 C CNN
 F 1 "IN" V 1300 4350 50  0000 C CNN
-F 2 "" H 1200 4350 50  0000 C CNN
+F 2 "Pin_Headers:Pin_Header_Straight_1x02_Pitch2.54mm" H 1200 4350 50  0001 C CNN
 F 3 "" H 1200 4350 50  0000 C CNN
 	1    1200 4350
@@
 	1500 4400 1500 4500
 $Comp
-L GND #PWR3
+L GND #PWR010
 U 1 1 5AD2F7B4
 P 1500 4500
-F 0 "#PWR3" H 1500 4250 50  0001 C CNN
+F 0 "#PWR010" H 1500 4250 50  0001 C CNN
 F 1 "GND" H 1500 4350 50  0000 C CNN
 F 2 "" H 1500 4500 50  0000 C CNN
@@
 F 0 "P4" H 10700 4500 50  0000 C CNN
 F 1 "OUT" V 10800 4350 50  0000 C CNN
-F 2 "" H 10700 4350 50  0000 C CNN
+F 2 "Pin_Headers:Pin_Header_Straight_1x02_Pitch2.54mm" H 10700 4350 50  0001 C CNN
 F 3 "" H 10700 4350 50  0000 C CNN
 	1    10700 4350
@@
 OUT
 $Comp
-L GND #PWR14
+L GND #PWR011
 U 1 1 5AD30334
 P 10400 4500
-F 0 "#PWR14" H 10400 4250 50  0001 C CNN
+F 0 "#PWR011" H 10400 4250 50  0001 C CNN
 F 1 "GND" H 10400 4350 50  0000 C CNN
 F 2 "" H 10400 4500 50  0000 C CNN
@@
 F 0 "P3" H 1200 6000 50  0000 C CNN
 F 1 "Takt" V 1300 5800 50  0000 C CNN
-F 2 "" H 1200 5800 50  0000 C CNN
+F 2 "Pin_Headers:Pin_Header_Straight_1x03_Pitch2.54mm" H 1200 5800 50  0001 C CNN
 F 3 "" H 1200 5800 50  0000 C CNN
 	1    1200 5800
@@
 $EndComp
 $Comp
-L GND #PWR4
+L GND #PWR012
 U 1 1 5AD31244
 P 1600 6100
-F 0 "#PWR4" H 1600 5850 50  0001 C CNN
+F 0 "#PWR012" H 1600 5850 50  0001 C CNN
 F 1 "GND" H 1600 5950 50  0000 C CNN
 F 2 "" H 1600 6100 50  0000 C CNN
@@
 F 0 "P1" H 1200 1900 50  0000 C CNN
 F 1 "Power" V 1300 1750 50  0000 C CNN
-F 2 "" H 1200 1750 50  0000 C CNN
+F 2 "Pin_Headers:Pin_Header_Straight_1x02_Pitch2.54mm" H 1200 1750 50  0001 C CNN
 F 3 "" H 1200 1750 50  0000 C CNN
 	1    1200 1750
@@
 $EndComp
 $Comp
-L GND #PWR2
+L GND #PWR013
 U 1 1 5AD32AD2
 P 1500 1900
-F 0 "#PWR2" H 1500 1650 50  0001 C CNN
+F 0 "#PWR013" H 1500 1650 50  0001 C CNN
 F 1 "GND" H 1500 1750 50  0000 C CNN
 F 2 "" H 1500 1900 50  0000 C CNN
@@
 	1500 1800 1500 1900
 $Comp
-L +5V #PWR1
+L +5V #PWR014
 U 1 1 5AD32D6F
 P 1500 1600
-F 0 "#PWR1" H 1500 1450 50  0001 C CNN
+F 0 "#PWR014" H 1500 1450 50  0001 C CNN
 F 1 "+5V" H 1500 1740 50  0000 C CNN
 F 2 "" H 1500 1600 50  0000 C CNN
@@
 Wire Wire Line
 	1500 1700 1500 1600
+$Comp
+L TRANSFORMER_1P_2S_2 T1
+U 1 1 5AD259DF
+P 3100 4300
+F 0 "T1" H 3100 4800 50  0000 C CNN
+F 1 "Übertrager" H 3100 3800 50  0000 C CNN
+F 2 "HF_Transformers:T-622" H 3100 4300 50  0001 C CNN
+F 3 "" H 3100 4300 50  0000 C CNN
+	1    3100 4300
+	1    0    0    -1
+$EndComp
 $EndSCHEMATC

Commit message: Schaltplan Rev D, Layout Rev A
Parts:
- C1: footprint Capacitors_THT:C_Radial_D6.3_L11.2_P2.5 -> Discret:C1V7H_2
Connections:
- net IN1 is gone; now on net SW1: U1.13 (OE)
- net GND: now also T2.1 (AA); no longer T2.6 (AB)
- net OUT: now also T2.6 (AB); no longer T2.1 (AA)
- net SW1: now also U1.4 (OE); no longer U1.1 (OE)
- net SW2: now also U1.1 (OE), U1.10 (OE); no longer U1.10 (OE), U1.4 (OE)
- net at T1.5 (SD), U1.12 (A): now also U1.2 (A); no longer U1.9 (A)
- new net: T1.3 (SA), U1.5 (A), U1.9 (A)
- new net: T2.5 (SD), U1.3 (B), U1.6 (B)
- new net: T2.3 (SA), U1.11 (B), U1.8 (B)
Changed lines of the file:
@@
 Sheet 1 1
 Title "Schaltmischer"
-Date "2018-04-14"
-Rev "C"
+Date "2018-04-15"
+Rev "D"
 Comp "Jonas Gappert"
 Comment1 ""
@@
 $Comp
 L FST3125 U1
-U 1 1 5AD24E27
+U 2 1 5AD24E27
 P 5500 2400
 F 0 "U1" H 5500 2650 60  0000 C CNN
@@
 F 2 "Housings_SOIC:SOIC-14_3.9x8.7mm_Pitch1.27mm" H 5500 2400 60  0001 C CNN
 F 3 "" H 5500 2400 60  0001 C CNN
-	1    5500 2400
+	2    5500 2400
 	1    0    0    -1
 $EndComp
 $Comp
 L FST3125 U1
-U 2 1 5AD24EC6
+U 3 1 5AD24EC6
 P 5500 3400
 F 0 "U1" H 5500 3650 60  0000 C CNN
@@
 F 2 "Housings_SOIC:SOIC-14_3.9x8.7mm_Pitch1.27mm" H 5500 3400 60  0001 C CNN
 F 3 "" H 5500 3400 60  0001 C CNN
-	2    5500 3400
+	3    5500 3400
 	1    0    0    -1
 $EndComp
 $Comp
 L FST3125 U1
-U 3 1 5AD24F31
+U 1 1 5AD24F31
 P 5500 4600
 F 0 "U1" H 5500 4850 60  0000 C CNN
@@
 F 2 "Housings_SOIC:SOIC-14_3.9x8.7mm_Pitch1.27mm" H 5500 4600 60  0001 C CNN
 F 3 "" H 5500 4600 60  0001 C CNN
-	3    5500 4600
-	1    0    0    -1
-$EndComp
-$Comp
-L FST3125 U1
-U 4 1 5AD24F98
-P 5500 5600
-F 0 "U1" H 5500 5850 60  0000 C CNN
-F 1 "FST3125" H 5600 5150 60  0000 C CNN
-F 2 "Housings_SOIC:SOIC-14_3.9x8.7mm_Pitch1.27mm" H 5500 5600 60  0001 C CNN
-F 3 "" H 5500 5600 60  0001 C CNN
-	4    5500 5600
+	1    5500 4600
 	1    0    0    -1
 $EndComp
@@
 SW1
 Text GLabel 5000 5600 0    60   Input ~ 0
-IN1
+SW1
 Wire Wire Line
 	5200 2700 4700 2700
@@
 F 3 "" H 8700 4300 50  0000 C CNN
 	1    8700 4300
-	-1   0    0    -1
+	-1   0    0    1
 $EndComp
 Wire Wire Line
@@
 F 0 "C1" H 3225 2350 50  0000 L CNN
 F 1 "10µ" H 3225 2150 50  0000 L CNN
-F 2 "Capacitors_THT:C_Radial_D6.3_L11.2_P2.5" H 3238 2100 50  0001 C CNN
+F 2 "Discret:C1V7H_2" H 3238 2100 50  0001 C CNN
 F 3 "" H 3200 2250 50  0000 C CNN
 	1    3200 2250
@@
 	1    0    0    -1
 $EndComp
+$Comp
+L FST3125 U1
+U 4 1 5AD24F98
+P 5500 5600
+F 0 "U1" H 5500 5850 60  0000 C CNN
+F 1 "FST3125" H 5600 5150 60  0000 C CNN
+F 2 "Housings_SOIC:SOIC-14_3.9x8.7mm_Pitch1.27mm" H 5500 5600 60  0001 C CNN
+F 3 "" H 5500 5600 60  0001 C CNN
+	4    5500 5600
+	1    0    0    -1
+$EndComp

Commit message: save before gnd floating
Parts:
- added P5, P6, P7, P8: GND, Mounting_Holes:MountingHole_3.2mm_M3_Pad_Via, symbol TEST
Connections:
- net GND: now also P5.1, P6.1, P7.1, P8.1
Other:
- note added: "Befestigungsbohrungen"
Changed lines of the file:
@@
 	8200 4400 8300 4400
 $Comp
-L GND #PWR01
+L GND #PWR6
 U 1 1 5AD25ECC
 P 2500 4700
-F 0 "#PWR01" H 2500 4450 50  0001 C CNN
+F 0 "#PWR6" H 2500 4450 50  0001 C CNN
 F 1 "GND" H 2500 4550 50  0000 C CNN
 F 2 "" H 2500 4700 50  0000 C CNN
@@
 $EndComp
 $Comp
-L GND #PWR02
+L GND #PWR12
 U 1 1 5AD25F11
 P 9300 4700
-F 0 "#PWR02" H 9300 4450 50  0001 C CNN
+F 0 "#PWR12" H 9300 4450 50  0001 C CNN
 F 1 "GND" H 9300 4550 50  0000 C CNN
 F 2 "" H 9300 4700 50  0000 C CNN
@@
 Connection ~ 3600 4300
 $Comp
-L GND #PWR03
+L GND #PWR10
 U 1 1 5AD27FC4
 P 3800 5400
-F 0 "#PWR03" H 3800 5150 50  0001 C CNN
+F 0 "#PWR10" H 3800 5150 50  0001 C CNN
 F 1 "GND" H 3800 5250 50  0000 C CNN
 F 2 "" H 3800 5400 50  0000 C CNN
@@
 $EndComp
 $Comp
-L GND #PWR04
+L GND #PWR11
 U 1 1 5AD283A9
 P 8000 5400
-F 0 "#PWR04" H 8000 5150 50  0001 C CNN
+F 0 "#PWR11" H 8000 5150 50  0001 C CNN
 F 1 "GND" H 8000 5250 50  0000 C CNN
 F 2 "" H 8000 5400 50  0000 C CNN
@@
 Connection ~ 3200 1800
 $Comp
-L GND #PWR05
+L GND #PWR7
 U 1 1 5AD2A7C7
 P 2600 2500
-F 0 "#PWR05" H 2600 2250 50  0001 C CNN
+F 0 "#PWR7" H 2600 2250 50  0001 C CNN
 F 1 "GND" H 2600 2350 50  0000 C CNN
 F 2 "" H 2600 2500 50  0000 C CNN
@@
 $EndComp
 $Comp
-L GND #PWR06
+L GND #PWR9
 U 1 1 5AD2A809
 P 3200 2500
-F 0 "#PWR06" H 3200 2250 50  0001 C CNN
+F 0 "#PWR9" H 3200 2250 50  0001 C CNN
 F 1 "GND" H 3200 2350 50  0000 C CNN
 F 2 "" H 3200 2500 50  0000 C CNN
@@
 Connection ~ 2900 1800
 $Comp
-L +5V #PWR07
+L +5V #PWR8
 U 1 1 5AD2B086
 P 2900 1100
-F 0 "#PWR07" H 2900 950 50  0001 C CNN
+F 0 "#PWR8" H 2900 950 50  0001 C CNN
 F 1 "+5V" H 2900 1240 50  0000 C CNN
 F 2 "" H 2900 1100 50  0000 C CNN
@@
 	2900 1100 2900 1200
 $Comp
-L GND #PWR08
+L GND #PWR14
 U 1 1 5AD2BFA4
 P 9700 2700
-F 0 "#PWR08" H 9700 2450 50  0001 C CNN
+F 0 "#PWR14" H 9700 2450 50  0001 C CNN
 F 1 "GND" H 9700 2550 50  0000 C CNN
 F 2 "" H 9700 2700 50  0000 C CNN
@@
 $EndComp
 $Comp
-L +5V #PWR09
+L +5V #PWR13
 U 1 1 5AD2C04B
 P 9700 1300
-F 0 "#PWR09" H 9700 1150 50  0001 C CNN
+F 0 "#PWR13" H 9700 1150 50  0001 C CNN
 F 1 "+5V" H 9700 1440 50  0000 C CNN
 F 2 "" H 9700 1300 50  0000 C CNN
@@
 	1500 4400 1500 4500
 $Comp
-L GND #PWR010
+L GND #PWR3
 U 1 1 5AD2F7B4
 P 1500 4500
-F 0 "#PWR010" H 1500 4250 50  0001 C CNN
+F 0 "#PWR3" H 1500 4250 50  0001 C CNN
 F 1 "GND" H 1500 4350 50  0000 C CNN
 F 2 "" H 1500 4500 50  0000 C CNN
@@
 OUT
 $Comp
-L GND #PWR011
+L GND #PWR15
 U 1 1 5AD30334
 P 10400 4500
-F 0 "#PWR011" H 10400 4250 50  0001 C CNN
+F 0 "#PWR15" H 10400 4250 50  0001 C CNN
 F 1 "GND" H 10400 4350 50  0000 C CNN
 F 2 "" H 10400 4500 50  0000 C CNN
@@
 $EndComp
 $Comp
-L GND #PWR012
+L GND #PWR4
 U 1 1 5AD31244
 P 1600 6100
-F 0 "#PWR012" H 1600 5850 50  0001 C CNN
+F 0 "#PWR4" H 1600 5850 50  0001 C CNN
 F 1 "GND" H 1600 5950 50  0000 C CNN
 F 2 "" H 1600 6100 50  0000 C CNN
@@
 $EndComp
 $Comp
-L GND #PWR013
+L GND #PWR2
 U 1 1 5AD32AD2
 P 1500 1900
-F 0 "#PWR013" H 1500 1650 50  0001 C CNN
+F 0 "#PWR2" H 1500 1650 50  0001 C CNN
 F 1 "GND" H 1500 1750 50  0000 C CNN
 F 2 "" H 1500 1900 50  0000 C CNN
@@
 	1500 1800 1500 1900
 $Comp
-L +5V #PWR014
+L +5V #PWR1
 U 1 1 5AD32D6F
 P 1500 1600
-F 0 "#PWR014" H 1500 1450 50  0001 C CNN
+F 0 "#PWR1" H 1500 1450 50  0001 C CNN
 F 1 "+5V" H 1500 1740 50  0000 C CNN
 F 2 "" H 1500 1600 50  0000 C CNN
@@
 	1    0    0    -1
 $EndComp
+$Comp
+L TEST P5
+U 1 1 5AD32637
+P 1300 7000
+F 0 "P5" H 1300 7300 50  0000 C BNN
+F 1 "GND" H 1300 7250 50  0000 C CNN
+F 2 "Mounting_Holes:MountingHole_3.2mm_M3_Pad_Via" H 1300 7000 50  0001 C CNN
+F 3 "" H 1300 7000 50  0000 C CNN
+	1    1300 7000
+	1    0    0    -1
+$EndComp
+$Comp
+L TEST P6
+U 1 1 5AD32C6F
+P 1500 7000
+F 0 "P6" H 1500 7300 50  0000 C BNN
+F 1 "GND" H 1500 7250 50  0000 C CNN
+F 2 "Mounting_Holes:MountingHole_3.2mm_M3_Pad_Via" H 1500 7000 50  0001 C CNN
+F 3 "" H 1500 7000 50  0000 C CNN
+	1    1500 7000
+	1    0    0    -1
+$EndComp
+$Comp
+L TEST P7
+U 1 1 5AD32CC0
+P 1700 7000
+F 0 "P7" H 1700 7300 50  0000 C BNN
+F 1 "GND" H 1700 7250 50  0000 C CNN
+F 2 "Mounting_Holes:MountingHole_3.2mm_M3_Pad_Via" H 1700 7000 50  0001 C CNN
+F 3 "" H 1700 7000 50  0000 C CNN
+	1    1700 7000
+	1    0    0    -1
+$EndComp
+$Comp
+L TEST P8
+U 1 1 5AD32D0C
+P 1900 7000
+F 0 "P8" H 1900 7300 50  0000 C BNN
+F 1 "GND" H 1900 7250 50  0000 C CNN
+F 2 "Mounting_Holes:MountingHole_3.2mm_M3_Pad_Via" H 1900 7000 50  0001 C CNN
+F 3 "" H 1900 7000 50  0000 C CNN
+	1    1900 7000
+	1    0    0    -1
+$EndComp
+$Comp
+L GND #PWR5
+U 1 1 5AD32DC8
+P 1600 7200
+F 0 "#PWR5" H 1600 6950 50  0001 C CNN
+F 1 "GND" H 1600 7050 50  0000 C CNN
+F 2 "" H 1600 7200 50  0000 C CNN
+F 3 "" H 1600 7200 50  0000 C CNN
+	1    1600 7200
+	1    0    0    -1
+$EndComp
+Wire Wire Line
+	1300 7000 1300 7100
+Wire Wire Line
+	1300 7100 1900 7100
+Wire Wire Line
+	1900 7100 1900 7000
+Wire Wire Line
+	1600 7100 1600 7200
+Connection ~ 1600 7100
+Wire Wire Line
+	1500 7000 1500 7100
+Connection ~ 1500 7100
+Wire Wire Line
+	1700 7000 1700 7100
+Connection ~ 1700 7100
+Text Notes 2100 7000 0    60   ~ 0
+Befestigungsbohrungen
 $EndSCHEMATC

Commit message: save after gnd floating
Connections:
- net GND: now also T2.6 (AB); no longer T2.1 (AA)
- net OUT: now also T2.1 (AA); no longer T2.6 (AB)
- net at U1.3 (B), U1.6 (B): now also T2.3 (SA); no longer T2.5 (SD)
- net at U1.11 (B), U1.8 (B): now also T2.5 (SD); no longer T2.3 (SA)
Changed lines of the file:
@@
 F 3 "" H 8700 4300 50  0000 C CNN
 	1    8700 4300
-	-1   0    0    1
+	-1   0    0    -1
 $EndComp
 Wire Wire Line
